File: Hardware/SelectaAutomatKeyPad/SelectaAutomatKeyPad.kicad_pcb (KiCad board)
At the start: 2 copper layers, 73.5 x 104 mm, 13 parts, among them J1 Conn_01x07_Male, SW1 TS-1003S-04326, SW10 TS-1003S-04326, SW11 TS-1003S-04326, SW12 TS-1003S-04326, SW2 TS-1003S-04326, SW3 TS-1003S-04326, SW4 TS-1003S-04326, SW5 TS-1003S-04326, SW6 TS-1003S-04326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

Commit message: wotk on lyout + doku
Parts:
- moved J1 1.76 mm to (129.1, 50.0)
Connections:
- SW12 pad 1: /1 -> /1A
- SW3 pad 1: /C -> /C1
- SW8 pad 1: /B -> /B1
- SW9 pad 1: /4 -> /4A
Routing:
- net /A: track 0.00 -> 206.8 mm
- net /B: track 0.00 -> 190.7 mm
- net /3: track 0.00 -> 158.3 mm
- net /2: track 0.00 -> 113.8 mm
- net /1: track 0.00 -> 111.7 mm
- net /4A: track 0.00 -> 65.9 mm
- net /C: track 0.00 -> 60.0 mm
- net /4: track 0.00 -> 46.2 mm
- net /2A: track 0.00 -> 26.8 mm
- net /1A: track 0.00 -> 20.4 mm
- net /C1: track 0.00 -> 9.05 mm
- net /B1: track 0.00 -> 8.86 mm
Other:
- board text added: "Designer: Edwin Koch"
- board text added: "Keypad 20230306"
- board text removed: "Keypad 20230304"

Commit message: created gerberfiles
Parts:
- added H1: MountingHole, MountingHole:MountingHole_2.1mm, F.Cu at (104.3, 145.7)
- added H2: MountingHole, MountingHole:MountingHole_2.1mm, F.Cu at (170.5, 147.0)
- added H3: MountingHole, MountingHole:MountingHole_2.1mm, F.Cu at (170.5, 49.0)
- added H4: MountingHole, MountingHole:MountingHole_2.1mm, F.Cu at (103.0, 49.0)
Routing:
- net /1: track 111.7 -> 110.0 mm
- net /A: track 206.8 -> 207.4 mm
Other:
- outline, holes or cut-outs redrawn
- board text added: "Keypad 20230326"
- board text removed: "Keypad 20230306"
