File: Hardware/SelectaAutomatKeyPad/SelectaAutomatKeyPad.kicad_sch (KiCad schematic)
At the start: 13 parts

Commit message: work on layout
Parts:
- removed SW? (x12): SW_MEC_5E, symbol Switch:SW_MEC_5E
- added SW1, SW10, SW11, SW12, SW2, SW3, SW4, SW5, SW6, SW7, SW8, SW9: TS-1003S-04326, 870_Button_SMD:TS-1003S, symbol 870_Button_SMD:TS-1003S-04326
- J1: renamed from J?; footprint Connector_PinHeader_1.00mm:PinHeader_1x07_P1.00mm_Horizontal -> Connector_PinHeader_2.54mm:PinHeader_1x07_P2.54mm_Horizontal
Connections:
- net 1: now also SW12.1, SW4.4 (A), SW8.4 (A)
- net 2: now also SW10.4 (A), SW3.4 (A), SW7.4 (A)
- net 3: now also SW11.4 (A), SW2.4 (A), SW6.1
- net 4: now also SW1.1, SW5.4 (A), SW9.1
- net A: now also SW10.1, SW11.1, SW12.4 (A), SW9.4 (A)
- net B: now also SW5.1, SW6.4 (A), SW7.1, SW8.1
- net C: now also SW1.4 (A), SW2.1, SW3.1, SW4.1

Commit message: wotk on lyout + doku
Connections:
- net 1: no longer SW12.1
- net 2: now also SW7.3 (K); no longer SW10.4 (A), SW7.4 (A)
- net 4: no longer SW5.4 (A), SW9.1
- net B: no longer SW8.1
- net C: no longer SW3.1
- net B1: now reaches SW7.2
- net B1: now also SW8.1
- net C1: now reaches SW2.2
- net C1: now also SW3.1
- net 1A: now reaches SW8.3 (K)
- net 1A: now also SW12.1
- net 4A: now reaches SW1.2
- net 4A: now also SW5.4 (A), SW9.1
- new net 2A: SW10.4 (A), SW7.4 (A)
Other:
- title: (none) -> Keypad

Commit message: created gerberfiles
Parts:
- added H1, H2, H3, H4: MountingHole, MountingHole:MountingHole_2.1mm, symbol Mechanical:MountingHole
Changed lines of the file:
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@@
   (title_block
     (title "Keypad")
-    (date "2023-03-06")
+    (date "2023-03-26")
     (rev "20230306")
     (comment 1 "Edwin Koch")
@@
     (pin "3")
     (pin "4")
+  )
+  (symbol (lib_id "Mechanical:MountingHole") (at 139.7 177.8 0) (unit 1)
+    (in_bom yes) (on_board yes) (fields_autoplaced)
+    (property "Reference" "H2" (id 0) (at 142.24 176.5299 0)
+      (effects (font (size 1.27 1.27)) (justify left))
+    )
+    (property "Value" "MountingHole" (id 1) (at 142.24 179.0699 0)
+      (effects (font (size 1.27 1.27)) (justify left))
+    )
+    (property "Footprint" "MountingHole:MountingHole_2.1mm" (id 2) (at 139.7 177.8 0)
+      (effects (font (size 1.27 1.27)) hide)
+    )
+    (property "Datasheet" "~" (id 3) (at 139.7 177.8 0)
+      (effects (font (size 1.27 1.27)) hide)
+    )
+  )
+  (symbol (lib_id "Mechanical:MountingHole") (at 139.7 184.15 0) (unit 1)
+    (in_bom yes) (on_board yes) (fields_autoplaced)
+    (property "Reference" "H3" (id 0) (at 142.24 182.8799 0)
+      (effects (font (size 1.27 1.27)) (justify left))
+    )
+    (property "Value" "MountingHole" (id 1) (at 142.24 185.4199 0)
+      (effects (font (size 1.27 1.27)) (justify left))
+    )
+    (property "Footprint" "MountingHole:MountingHole_2.1mm" (id 2) (at 139.7 184.15 0)
+      (effects (font (size 1.27 1.27)) hide)
+    )
+    (property "Datasheet" "~" (id 3) (at 139.7 184.15 0)
+      (effects (font (size 1.27 1.27)) hide)
+    )
   )
   (symbol (lib_id "870_Button_SMD:TS-1003S-04326") (at 114.3 101.6 0) (unit 1)
@@
     (pin "4")
   )
+  (symbol (lib_id "Mechanical:MountingHole") (at 139.7 171.45 0) (unit 1)
+    (in_bom yes) (on_board yes) (fields_autoplaced)
+    (property "Reference" "H1" (id 0) (at 142.24 170.1799 0)
+      (effects (font (size 1.27 1.27)) (justify left))
+    )
+    (property "Value" "MountingHole" (id 1) (at 142.24 172.7199 0)
+      (effects (font (size 1.27 1.27)) (justify left))
+    )
+    (property "Footprint" "MountingHole:MountingHole_2.1mm" (id 2) (at 139.7 171.45 0)
+      (effects (font (size 1.27 1.27)) hide)
+    )
+    (property "Datasheet" "~" (id 3) (at 139.7 171.45 0)
+      (effects (font (size 1.27 1.27)) hide)
+    )
+  )
   (symbol (lib_id "870_Button_SMD:TS-1003S-04326") (at 165.1 76.2 0) (unit 1)
     (in_bom yes) (on_board yes) (fields_autoplaced)
@@
     (pin "4")
   )
+  (symbol (lib_id "Mechanical:MountingHole") (at 139.7 190.5 0) (unit 1)
+    (in_bom yes) (on_board yes) (fields_autoplaced)
+    (property "Reference" "H4" (id 0) (at 142.24 189.2299 0)
+      (effects (font (size 1.27 1.27)) (justify left))
+    )
+    (property "Value" "MountingHole" (id 1) (at 142.24 191.7699 0)
+      (effects (font (size 1.27 1.27)) (justify left))
+    )
+    (property "Footprint" "MountingHole:MountingHole_2.1mm" (id 2) (at 139.7 190.5 0)
+      (effects (font (size 1.27 1.27)) hide)
+    )
+    (property "Datasheet" "~" (id 3) (at 139.7 190.5 0)
+      (effects (font (size 1.27 1.27)) hide)
+    )
+  )
   (symbol (lib_id "870_Button_SMD:TS-1003S-04326") (at 139.7 152.4 0) (unit 1)
     (in_bom yes) (on_board yes) (fields_autoplaced)
@@
   )
   (symbol_instances
+    (path "/bac26624-7015-4c97-ab11-33bb9a36bdb1"
+      (reference "H1") (unit 1) (value "MountingHole") (footprint "MountingHole:MountingHole_2.1mm")
+    )
+    (path "/1a4b9d7b-c263-4312-b020-5f270732b097"
+      (reference "H2") (unit 1) (value "MountingHole") (footprint "MountingHole:MountingHole_2.1mm")
+    )
+    (path "/1d560296-72fc-42d8-bf15-aea12bb584ef"
+      (reference "H3") (unit 1) (value "MountingHole") (footprint "MountingHole:MountingHole_2.1mm")
+    )
+    (path "/e68e90c5-5e22-492f-b218-e6158f0a4e22"
+      (reference "H4") (unit 1) (value "MountingHole") (footprint "MountingHole:MountingHole_2.1mm")
+    )
     (path "/24bf3703-ca0e-498d-8754-0db3975afcb8"
       (reference "J1") (unit 1) (value "Conn_01x07_Male") (footprint "Connector_PinHeader_2.54mm:PinHeader_1x07_P2.54mm_Horizontal")
